Commit message: before changing the drive controller in 4 wheeled robot

File: robot_model_pkg/urdf/robot.xacro (robot description, xacro)
@@ -1,243 +1,265 @@
 <?xml version="1.0"?>
-<robot name="differential_drive_robot" xmlns:xacro="https://www.ros.org/wiki/xacro">
-<!-- base dimensions -->
-<xacro:property name="base_link_x_dim" value="1"/>
-<xacro:property name="base_link_y_dim" value="0.6"/>
-<xacro:property name="base_link_z_dim" value="0.3"/>
-<!-- Wheel dimensions -->
-<xacro:property name="wheel_link_radius" value="0.15"/>
-<xacro:property name="wheel_link_length" value="0.1"/>
-<xacro:property name="wheel_link_z_location" value="-0.1"/>
-<!-- Material density -->
-<xacro:property name="base_density" value="2710.0"/>
-<xacro:property name="wheel_density" value="2710.0"/>
-<!-- Pi constant -->
-<xacro:property name="pi_const" value="3.14159265"/>
-<!--Robot base and wheel mass -->
-<xacro:property name="base_mass" value="${base_density*base_link_x_dim*base_link_y_dim*base_link_z_dim}"/>
-<xacro:property name="wheel_mass" value="${wheel_density*pi_const*wheel_link_radius*wheel_link_radius*wheel_link_length}"/>
-<!-- Compute inertia terms -->
-<xacro:property name="ixx" value="${(1.0/12.0) * base_mass * (base_link_y_dim**2 + base_link_z_dim**2)}"/>
-<xacro:property name="iyy" value="${(1.0/12.0) * base_mass * (base_link_x_dim**2 + base_link_z_dim**2)}"/>
-<xacro:property name="izz" value="${(1.0/12.0) * base_mass * (base_link_x_dim**2 + base_link_y_dim**2)}"/>
-<!-- Moments of inertia of the wheel -->
-<xacro:property name="Iz_wheel" value="${0.5*wheel_mass*wheel_link_radius*wheel_link_radius}"/>
-<xacro:property name="I_wheel" value="${(1.0/12.0)*wheel_mass*(3.0*wheel_link_radius*wheel_link_radius+wheel_link_length*wheel_link_length)}" />
-<!-- This macro defines the complete inertial section of the wheel -->
-<xacro:macro name="inertia_wheel">
-	<inertial>
-	<origin rpy="0 0 0" xyz="0 0 0"/>
-	<mass value="${wheel_mass}"/>
-	<inertia ixx="${I_wheel}" ixy="0.0" ixz="0.0" iyy="${I_wheel}" iyz="0.0" izz="${Iz_wheel}"/>
-	</inertial>
-</xacro:macro>
-<!-- we include the file that defines extra Gazebo options and motion control driver -->
-<xacro:include filename="$(find robot_model_pkg)/urdf/robot.gazebo" />
-<!-- Links and Joints -->
-<!--base link-->
-<link name="base_link">
-	<visual>
-		<geometry>
-			<box size="${base_link_x_dim} ${base_link_y_dim} ${base_link_z_dim/2}" />
-		</geometry>
-	<origin rpy="0 0 0" xyz="0 0 0"/>
-	</visual>
-	<collision>
-		<geometry>
-			<box size="${base_link_x_dim} ${base_link_y_dim} ${base_link_z_dim}"/>
-		</geometry>
-		<origin rpy="0 0 0" xyz="0 0 0"/>
-	</collision>
-	<inertial>
-		<origin rpy="0 0 0" xyz="0 0 0"/>
-		<mass value="${base_mass}"/>
-		<inertia ixx="${ixx}" ixy="0" ixz="0" iyy="${iyy}" iyz="0" izz="${izz}"/>
-	</inertial>
-</link>
-<!-- Kinect Sensor joint -->
-<joint name="camera_joint" type="fixed">
-	<parent link="base_link"/>
-	<child link="camera_link"/>
-	<origin xyz="${base_link_x_dim/2} 0 ${base_link_z_dim/3}" rpy="0 0 0"/>
-</joint>
-<link name="camera_link">
-	<visual>
-		<origin rpy="0 0 0" xyz="0 0 0"/>
-		<geometry>
-			<box size="0.3 0.4 0.1"/>
-		</geometry>
-	</visual>
-	<collision>
-		<geometry>
+<robot name="differential_drive_robot"
+	xmlns:xacro="https://www.ros.org/wiki/xacro">
+	<!-- base dimensions -->
+	<xacro:property name="base_link_x_dim" value="1"/>
+	<xacro:property name="base_link_y_dim" value="0.6"/>
+	<xacro:property name="base_link_z_dim" value="0.3"/>
+	<!-- Wheel dimensions -->
+	<xacro:property name="wheel_link_radius" value="0.15"/>
+	<xacro:property name="wheel_link_length" value="0.1"/>
+	<xacro:property name="wheel_link_z_location" value="-0.1"/>
+	<!-- Material density -->
+	<xacro:property name="base_density" value="2710.0"/>
+	<xacro:property name="wheel_density" value="2710.0"/>
+	<!-- Pi constant -->
+	<xacro:property name="pi_const" value="3.14159265"/>
+	<!--Robot base and wheel mass -->
+	<xacro:property name="base_mass" value="${base_density*base_link_x_dim*base_link_y_dim*base_link_z_dim}"/>
+	<xacro:property name="wheel_mass" value="${wheel_density*pi_const*wheel_link_radius*wheel_link_radius*wheel_link_length}"/>
+	<!-- Compute inertia terms -->
+	<xacro:property name="ixx" value="${(1.0/12.0) * base_mass * (base_link_y_dim**2 + base_link_z_dim**2)}"/>
+	<xacro:property name="iyy" value="${(1.0/12.0) * base_mass * (base_link_x_dim**2 + base_link_z_dim**2)}"/>
+	<xacro:property name="izz" value="${(1.0/12.0) * base_mass * (base_link_x_dim**2 + base_link_y_dim**2)}"/>
+	<!-- Moments of inertia of the wheel -->
+	<xacro:property name="Iz_wheel" value="${0.5*wheel_mass*wheel_link_radius*wheel_link_radius}"/>
+	<xacro:property name="I_wheel" value="${(1.0/12.0)*wheel_mass*(3.0*wheel_link_radius*wheel_link_radius+wheel_link_length*wheel_link_length)}" />
+	<!-- This macro defines the complete inertial section of the wheel -->
+	<xacro:macro name="inertia_wheel">
+		<inertial>
+			<origin rpy="0 0 0" xyz="0 0 0"/>
+			<mass value="${wheel_mass}"/>
+			<inertia ixx="${I_wheel}" ixy="0.0" ixz="0.0" iyy="${I_wheel}" iyz="0.0" izz="${Iz_wheel}"/>
+		</inertial>
+	</xacro:macro>
+	<!-- we include the file that defines extra Gazebo options and motion control driver -->
+	<xacro:include filename="$(find robot_model_pkg)/urdf/robot.gazebo" />
+	<!-- Links and Joints -->
+	<!--base link-->
+	<link name="base_link">
+		<visual>
+			<geometry>
+				<box size="${base_link_x_dim} ${base_link_y_dim} ${base_link_z_dim/2}" />
+			</geometry>
+			<origin rpy="0 0 0" xyz="0 0 0"/>
+		</visual>
+		<collision>
+			<geometry>
+				<box size="${base_link_x_dim} ${base_link_y_dim} ${base_link_z_dim}"/>
+			</geometry>
+			<origin rpy="0 0 0" xyz="0 0 0"/>
+		</collision>
+		<inertial>
+			<origin rpy="0 0 0" xyz="0 0 0"/>
+			<mass value="${base_mass}"/>
+			<inertia ixx="${ixx}" ixy="0" ixz="0" iyy="${iyy}" iyz="0" izz="${izz}"/>
+		</inertial>
+	</link>
+	<!-- Kinect Sensor joint -->
+	<joint name="camera_joint" type="fixed">
+		<parent link="base_link"/>
+		<child link="camera_link"/>
+		<origin xyz="${base_link_x_dim/2} 0 ${base_link_z_dim/3}" rpy="0 0 0"/>
+	</joint>
+	<link name="camera_link">
+		<visual>
+			<origin rpy="0 0 0" xyz="0 0 0"/>
+			<geometry>
 				<box size="0.3 0.4 0.1"/>
-		</geometry>
-		<origin rpy="0 0 0" xyz="0 0 0"/>
-	</collision>
-	<inertial>
-    <mass value="0.8"/>  <!-- Approximate weight of a Kinect -->
-    <origin xyz="0 0 0" rpy="0 0 0"/>
-    <inertia
-      ixx="0.002" ixy="0.0" ixz="0.0"
-      iyy="0.003" iyz="0.0"
-      izz="0.001"/>
-  </inertial>
-</link>
-<!-- Back Right wheel of the robot and the joint -->
-<joint name="wheel1_joint" type="continuous">
-	<parent link="base_link"/>
-	<child link="wheel1_link"/>
-	<origin xyz="${-base_link_x_dim/2+1.2*wheel_link_radius} ${-base_link_y_dim/2-wheel_link_length/2} ${wheel_link_z_location}" rpy="0 0 0"/>
-	<axis xyz="0 1 0"/>
-	<limit effort="1000" velocity="1000"/>
-	<dynamics damping="1.0" friction="1.0"/>
-</joint>
-<link name="wheel1_link">
-	<visual>
-		<origin rpy="1.570795 0 0" xyz="0 0 0"/>
-		<geometry>
-			<cylinder length="${wheel_link_length}" radius="${wheel_link_radius}"/>
-		</geometry>
-	</visual>
-	<collision>
-		<origin rpy="1.570795 0 0" xyz="0 0 0"/>
-		<geometry>
-			<cylinder length="${wheel_link_length}" radius="${wheel_link_radius}"/>
-		</geometry>
-	</collision>
-	<xacro:inertia_wheel />
-</link>
-<!-- Back Left wheel -->
-<joint name="wheel2_joint" type="continuous">
-	<parent link="base_link"/>
-	<child link="wheel2_link"/>
-	<origin xyz="${-base_link_x_dim/2+1.2*wheel_link_radius} ${base_link_y_dim/2+wheel_link_length/2} ${wheel_link_z_location}" rpy="0 0 0"/>
-	<axis xyz="0 1 0"/>
-	<limit effort="1000" velocity="1000"/>
-	<dynamics damping="1.0" friction="1.0"/>
-</joint>
-<link name="wheel2_link">
-	<visual>
-		<origin rpy="1.570795 0 0" xyz="0 0 0"/>
-		<geometry>
-			<cylinder length="${wheel_link_length}" radius="${wheel_link_radius}"/>
-		</geometry>
-	</visual>
-	<collision>
-		<origin rpy="1.570795 0 0" xyz="0 0 0"/>
-		<geometry>
-			<cylinder length="${wheel_link_length}" radius="${wheel_link_radius}"/>
-		</geometry>
-	</collision>
-	<xacro:inertia_wheel/>
-</link>
-<!-- Front Right Wheel -->
-<joint name="wheel3_joint" type="continuous">
-	<parent link="base_link"/>
-	<child link="wheel3_link"/>
-	<origin xyz="${base_link_x_dim/2-1.2*wheel_link_radius} ${-base_link_y_dim/2-wheel_link_length/2} ${wheel_link_z_location}" rpy="0 0 0"/>
-	<axis xyz="0 1 0"/>
-	<limit effort="1000" velocity="1000"/>
-	<dynamics damping="1.0" friction="1.0"/>
-</joint>
-<link name="wheel3_link">
-	<visual>
-		<origin rpy="1.570795 0 0" xyz="0 0 0"/>
-		<geometry>
-			<cylinder length="${wheel_link_length}" radius="${wheel_link_radius}"/>
-		</geometry>
-	</visual>
-	<collision>
-		<origin rpy="1.570795 0 0" xyz="0 0 0"/>
-			<geometry>
-				<cylinder length="${wheel_link_length}" radius="${wheel_link_radius}"/>
-			</geometry>
-	</collision>
-	<xacro:inertia_wheel/>
-</link>
-<!--Front Left-->
-<joint name="wheel4_joint" type="continuous">
-	<parent link="base_link"/>
-	<child link="wheel4_link"/>
-	<origin xyz="${base_link_x_dim/2-1.2*wheel_link_radius} ${base_link_y_dim/2+wheel_link_length/2} ${wheel_link_z_location}" rpy="0 0 0"/>
-	<axis xyz="0 1 0"/>
-	<limit effort="1000" velocity="1000"/>
-	<dynamics damping="1.0" friction="1.0"/>
-</joint>
-<link name="wheel4_link">
-	<visual>
-		<origin rpy="1.570795 0 0" xyz="0 0 0"/>
-		<geometry>
-			<cylinder length="${wheel_link_length}" radius="${wheel_link_radius}"/>
-		</geometry>
-	</visual>
-	<collision>
-		<origin rpy="1.570795 0 0" xyz="0 0 0"/>
-		<geometry>
-			<cylinder length="${wheel_link_length}" radius="${wheel_link_radius}"/>
-		</geometry>
-	</collision>
-	<xacro:inertia_wheel/>
-</link>
- <gazebo reference="camera_link">
-    <sensor type="multicamera" name="stereo_camera">
-      <update_rate>30.0</update_rate>
-      <camera name="left">
-        <horizontal_fov>1.3962634</horizontal_fov>
-        <image>
-          <width>800</width>
-          <height>800</height>
-          <format>R8G8B8</format>
-        </image>
-        <clip>
-          <near>0.02</near>
-          <far>300</far>
-        </clip>
-        <noise>
-          <type>gaussian</type>
-          <mean>0.0</mean>
-          <stddev>0.007</stddev>
-        </noise>
-      </camera>
-      <camera name="right">
-        <pose>0 -0.07 0 0 0 0</pose>
-        <horizontal_fov>1.3962634</horizontal_fov>
-        <image>
-          <width>800</width>
-          <height>800</height>
-          <format>R8G8B8</format>
-        </image>
-        <clip>
-          <near>0.02</near>
-          <far>300</far>
-        </clip>
-        <noise>
-          <type>gaussian</type>
-          <mean>0.0</mean>
-          <stddev>0.007</stddev>
-        </noise>
-      </camera>
-      <plugin name="stereo_camera_controller" filename="libgazebo_ros_multicamera.so">
-        <alwaysOn>true</alwaysOn>
-        <updateRate>1.0</updateRate>
-        <cameraName>stereo_camera</cameraName>
-		<imageTopicName>image_raw</imageTopicName>
-		<cameraInfoTopicName>camera_info</cameraInfoTopicName>
-		<frameName>camera_link</frameName>
-		<odometryTopic>/stereo_camera/odom</odometryTopic>
-		<rightImageTopicName>image_raw</rightImageTopicName>
-		<rightCameraInfoTopicName>camera_info</rightCameraInfoTopicName>
-		<rightFrameName>right_camera_optical_frame</rightFrameName>
-		<!-- Required by Gazebo -->
-		<covariance_x>0.0001</covariance_x>
-		<covariance_y>0.0001</covariance_y>
-		<covariance_yaw>0.01</covariance_yaw>
-        <hackBaseline>0.07</hackBaseline>
-        <distortionK1>0.00000001</distortionK1>
-      <distortionK2>0.00000001</distortionK2>
-      <distortionK3>0.00000001</distortionK3>
-      <distortionT1>0.00000001</distortionT1>
-      <distortionT2>0.00000001</distortionT2>
-      </plugin>
-    </sensor>
-  </gazebo>
+			</geometry>
+		</visual>
+		<collision>
+			<geometry>
+				<box size="0.3 0.4 0.1"/>
+			</geometry>
+			<origin rpy="0 0 0" xyz="0 0 0"/>
+		</collision>
+		<inertial>
+			<mass value="0.8"/>
+			<!-- Approximate weight of a Kinect -->
+			<origin xyz="0 0 0" rpy="0 0 0"/>
+			<inertia ixx="0.002" ixy="0.0" ixz="0.0" iyy="0.003" iyz="0.0" izz="0.001"/>
+		</inertial>
+	</link>
+	<!-- Back Right wheel of the robot and the joint -->
+	<joint name="wheel1_joint" type="continuous">
+		<parent link="base_link"/>
+		<child link="wheel1_link"/>
+		<origin xyz="${-base_link_x_dim/2+1.2*wheel_link_radius} ${-base_link_y_dim/2-wheel_link_length/2} ${wheel_link_z_location}" rpy="0 0 0"/>
+		<axis xyz="0 1 0"/>
+		<limit effort="1000" velocity="1000"/>
+		<dynamics damping="1.0" friction="1.0"/>
+	</joint>
+	<link name="wheel1_link">
+		<visual>
+			<origin rpy="1.570795 0 0" xyz="0 0 0"/>
+			<geometry>
+				<cylinder length="${wheel_link_length}" radius="${wheel_link_radius}"/>
+			</geometry>
+		</visual>
+		<collision>
+			<origin rpy="1.570795 0 0" xyz="0 0 0"/>
+			<geometry>
+				<cylinder length="${wheel_link_length}" radius="${wheel_link_radius}"/>
+			</geometry>
+		</collision>
+		<xacro:inertia_wheel />
+	</link>
+	<!-- Back Left wheel -->
+	<joint name="wheel2_joint" type="continuous">
+		<parent link="base_link"/>
+		<child link="wheel2_link"/>
+		<origin xyz="${-base_link_x_dim/2+1.2*wheel_link_radius} ${base_link_y_dim/2+wheel_link_length/2} ${wheel_link_z_location}" rpy="0 0 0"/>
+		<axis xyz="0 1 0"/>
+		<limit effort="1000" velocity="1000"/>
+		<dynamics damping="1.0" friction="1.0"/>
+	</joint>
+	<link name="wheel2_link">
+		<visual>
+			<origin rpy="1.570795 0 0" xyz="0 0 0"/>
+			<geometry>
+				<cylinder length="${wheel_link_length}" radius="${wheel_link_radius}"/>
+			</geometry>
+		</visual>
+		<collision>
+			<origin rpy="1.570795 0 0" xyz="0 0 0"/>
+			<geometry>
+				<cylinder length="${wheel_link_length}" radius="${wheel_link_radius}"/>
+			</geometry>
+		</collision>
+		<xacro:inertia_wheel/>
+	</link>
+	<!-- Front Right Wheel -->
+	<joint name="wheel3_joint" type="continuous">
+		<parent link="base_link"/>
+		<child link="wheel3_link"/>
+		<origin xyz="${base_link_x_dim/2-1.2*wheel_link_radius} ${-base_link_y_dim/2-wheel_link_length/2} ${wheel_link_z_location}" rpy="0 0 0"/>
+		<axis xyz="0 1 0"/>
+		<limit effort="1000" velocity="1000"/>
+		<dynamics damping="1.0" friction="1.0"/>
+	</joint>
+	<link name="wheel3_link">
+		<visual>
+			<origin rpy="1.570795 0 0" xyz="0 0 0"/>
+			<geometry>
+				<cylinder length="${wheel_link_length}" radius="${wheel_link_radius}"/>
+			</geometry>
+		</visual>
+		<collision>
+			<origin rpy="1.570795 0 0" xyz="0 0 0"/>
+			<geometry>
+				<cylinder length="${wheel_link_length}" radius="${wheel_link_radius}"/>
+			</geometry>
+		</collision>
+		<xacro:inertia_wheel/>
+	</link>
+	<!--Front Left-->
+	<joint name="wheel4_joint" type="continuous">
+		<parent link="base_link"/>
+		<child link="wheel4_link"/>
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